Commit message: done with center code for trimesh. some issues with collision in pybullet

File: pybullet_ur5_robotiq/urdfc/cube.urdf (robot description, URDF)
Before this commit: robot cube, 1 links, 0 joints
Links:
- link _name: geometry collision mesh filename=cube/tinker_vhacd.obj scale=0.001 0.001 0.0009; visual mesh filename=cube/tinker.obj scale=0.001 0.001 0.001
