Commit message: ignoring collision offset for now

File: pybullet_ur5_robotiq/urdfc/cuboid.urdf (robot description, URDF)
Before this commit: robot cuboid, 1 links, 0 joints
Links:
- link _name: geometry collision mesh filename=cuboid/tinker_vhacd.obj scale=0.00097 0.00097 0.00097; visual mesh filename=cuboid/tinker.obj scale=0.001 0.001 0.001

File: pybullet_ur5_robotiq/urdfc/cut_cuboid.urdf (robot description, URDF)
Before this commit: robot cut_cuboid, 1 links, 0 joints
Links:
- link _name: geometry collision mesh filename=cut_cuboid/tinker_vhacd.obj scale=0.00095 0.00095 0.0095; visual mesh filename=cut_cuboid/tinker.obj scale=0.001 0.001 0.001

Commit message: placement in trimesh done. some bug tof ix with closest point or plane creation

File: pybullet_ur5_robotiq/urdfc/cuboid.urdf (robot description, URDF)
Before this commit: robot cuboid, 1 links, 0 joints
Links:
- link _name: geometry collision mesh filename=cuboid/tinker_vhacd.obj scale=0.001 0.001 0.001; visual mesh filename=cuboid/tinker.obj scale=0.001 0.001 0.001

File: pybullet_ur5_robotiq/urdfc/cut_cuboid.urdf (robot description, URDF)
Before this commit: robot cut_cuboid, 1 links, 0 joints
Links:
- link _name: geometry collision mesh filename=cut_cuboid/tinker_vhacd.obj scale=0.001 0.001 0.001; visual mesh filename=cut_cuboid/tinker.obj scale=0.001 0.001 0.001
